Commit message: feat: table surface in urdf and update params for wbc
- add table surface in urdf model
- change parameters for updated whole body control

File: config/prismatic_fr3_duo.urdf.xacro (robot description, xacro)
@@ -23,3 +23,28 @@
       is_async="$(arg is_async)"
       thread_priority="$(arg thread_priority)"/>
+    <!-- Table surface-->
+    <link name="table_surface">
+        <visual>
+            <geometry>
+                <box size="1.0 2.0 0.01"/>
+            </geometry>
+            <material name="gray">
+                <color rgba="0.5 0.5 0.5 1.0"/>
+            </material>
+        </visual>
+        <collision>
+            <geometry>
+                <box size="1.0 2.0 0.01"/>
+            </geometry>
+        </collision>
+        <inertial>
+            <mass value="1.0"/>
+            <inertia ixx="0.01" ixy="0.0" ixz="0.0" iyy="0.01" iyz="0.0" izz="0.01"/>
+        </inertial>
+    </link>
+    <joint name="table_fix_joint" type="fixed">
+      <parent link="rail_link"/>
+      <child link="table_surface"/>
+      <origin xyz="0.5 0 0" rpy="0 0 0"/>
+    </joint>
 </robot>
